File: public/lights/orb-disc.kicad_pcb (KiCad board)
At the start: 2 copper layers, 70 x 70 mm, 66 parts, among them J1 riser in, J2 riser out, U1 AL8860 2200 K, U2 LMR16030, U3 AL8860 3000 K, U4 HDC3020

Commit message: lights: renders with bodies, pads rotated correctly, fab plots with outlines+designators
Co-Authored-By: Claude Fable 5 <noreply@anthropic.com>
Claude-Session: https://claude.ai/code/session_01KGs7HAmqeyDzRmkLXBVjfP
Parts:
- moved D3 0.36 mm to (119.9, 109.3), turned to 245.023 degrees
- moved L3 0.36 mm to (114.6, 116.4), turned to 221.748 degrees
- moved U3 0.18 mm to (108.3, 120.4), turned to 202.058 degrees
- moved U1 0.18 mm to (86.0, 116.9), turned to 140.394 degrees
- moved D2 0.16 mm to (80.3, 90.1), turned to 63.3812 degrees
- moved C_IN 0.16 mm to (87.8, 81.7), turned to 33.7199 degrees
- moved L2 0.16 mm to (100.4, 78.0), turned to 358.9 degrees
