File: public/lights/orb-disc.kicad_pcb (KiCad board)
At the start: 2 copper layers, 70 x 70 mm, 66 parts, among them J1 riser in, J2 riser out, U1 AL8860 2200 K, U2 LMR16030, U3 AL8860 3000 K, U4 HDC3020

Commit message: solar: h1 solar, OPT4048 sensor, drafted CAD drawings, plain-language sync note
Co-Authored-By: Claude Fable 5 <noreply@anthropic.com>
Claude-Session: https://claude.ai/code/session_01KGs7HAmqeyDzRmkLXBVjfP
Parts:
- added C_3V3: 1 uF, moistlab:C_0603, B.Cu at (110.1, 105.5)
- added C_SKY: 100 nF, moistlab:C_0402, F.Cu at (100.0, 104.0)
- added U5: OPT4048, moistlab:SOT-5X3-8, F.Cu at (100.0, 100.0)
- added U6: AP2112K-3.3, moistlab:SOT-23-5, B.Cu at (107.2, 109.0)
- moved R_SET_A 4.75 mm to (93.9, 109.8), turned to 147.982 degrees
- moved U4 4.75 mm to (98.2, 111.4), turned to 171.164 degrees
- moved R_SET_B 4.75 mm to (102.8, 111.1), turned to 194.346 degrees
