File: public/lights/orb-0-system.kicad_sch (KiCad schematic)
At the start: 6 parts

Commit message: solar: h1 solar, OPT4048 sensor, drafted CAD drawings, plain-language sync note
Co-Authored-By: Claude Fable 5 <noreply@anthropic.com>
Claude-Session: https://claude.ai/code/session_01KGs7HAmqeyDzRmkLXBVjfP
Other:
- note added: "CLIMATE: globes must breathe or they fog — vent + weep + coating are the defences, a humidity sensor per post proves they work (orb_climate.py)."
- note added: "POST BASE to its 4 DISCS: ONE cable of 7 conductors (+24V, GND, DATA, W_PWM_A, W_PWM_B, SDA, SCL); the discs daisy-chain — a chain has one input."
- note added: "Pin numbers are hidden on parts whose package pinout has NOT been transcribed. Only the 74AHCT125 and the OPT4048 have earned theirs."
- note added: "Provenance: ratings are [I] vendor web copy unless the part's note cites a document number — [M] only with a citation (first: U5/OPT4048, TI SBOSA84, 2026-08-03)."
- note removed: "CLIMATE: the globes must breathe or they fog. An ePTFE vent, a weep path and a coated board are the defences; the riser's I2C pair reaches a humidity sensor in the lowest globe of each post so that anyone can tell whether they are working. Heating is a supplement, not the mechanism — see orb_climate.py."
- note removed: "POST BASE to its 4 DISCS: ONE cable of 7 conductors (+24V, GND, DATA, W_PWM_A, W_PWM_B, SDA, SCL) to the first disc; the rest daisy-chain. It was drawn as four separate data lines until the disc's own J1->J2 chain contradicted it — a chain has one input."
- note removed: "Pin numbers are hidden on parts whose package pinout has NOT been transcribed. Only the 74AHCT125 shows its numbers."
- note removed: "Provenance: every rating on this sheet is [I] — vendor web copy or folklore. No transcription pass has happened."
Changed lines of the file:
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@@
 	(text "PACK to TAKEOFF: 160-233.6 VDC, 0.71 A worst, inches of cable, F_HV 2 A DC-rated to 1000 V." (exclude_from_sim no) (at 25.4 149.86 0) (effects (font (size 1.778 1.778)) (justify left)))
 	(text "TAKEOFF to each POST: 24 V regulated, 2.02 A nominal / 2.43 A at the 20 V design floor, 14 AWG buried 60 ft, F_P{1,2} 5 A blade (32 V rated — legal on THIS side only)." (exclude_from_sim no) (at 25.4 156.21 0) (effects (font (size 1.778 1.778)) (justify left)))
-	(text "POST BASE to its 4 DISCS: ONE cable of 7 conductors (+24V, GND, DATA, W_PWM_A, W_PWM_B, SDA, SCL) to the first disc; the rest daisy-chain. It was drawn as four separate data lines until the disc's own J1->J2 chain contradicted it — a chain has one input." (exclude_from_sim no) (at 25.4 162.56 0) (effects (font (size 1.778 1.778)) (justify left)))
+	(text "POST BASE to its 4 DISCS: ONE cable of 7 conductors (+24V, GND, DATA, W_PWM_A, W_PWM_B, SDA, SCL); the discs daisy-chain — a chain has one input." (exclude_from_sim no) (at 25.4 162.56 0) (effects (font (size 1.778 1.778)) (justify left)))
 	(text "WHOLE SYSTEM: 2 posts x 4 discs = 8 orb discs, 97.1 W flat out, 4.05 A of the converter's 6.5 A (62%)." (exclude_from_sim no) (at 25.4 168.91 0) (effects (font (size 1.778 1.778)) (justify left)))
 	(text "VOLTAGE DOMAINS: pack (lethal, one plate) / 24 V (everything buried and in-post) / 5 V (pixel rail, made per disc) / 3.3 V (ESP32 logic, re-driven to 5 V before it leaves the base)." (exclude_from_sim no) (at 25.4 175.26 0) (effects (font (size 1.778 1.778)) (justify left)))
-	(text "CLIMATE: the globes must breathe or they fog. An ePTFE vent, a weep path and a coated board are the defences; the riser's I2C pair reaches a humidity sensor in the lowest globe of each post so that anyone can tell whether they are working. Heating is a supplement, not the mechanism — see orb_climate.py." (exclude_from_sim no) (at 25.4 181.61 0) (effects (font (size 1.778 1.778)) (justify left)))
+	(text "CLIMATE: globes must breathe or they fog — vent + weep + coating are the defences, a humidity sensor per post proves they work (orb_climate.py)." (exclude_from_sim no) (at 25.4 181.61 0) (effects (font (size 1.778 1.778)) (justify left)))
 	(text "WHITE: two channels per disc, 2200 K and 3000 K, blended by the two dim lines. Same emitters and same watts as the single channel it replaced." (exclude_from_sim no) (at 25.4 187.96 0) (effects (font (size 1.778 1.778)) (justify left)))
 	(text "GENERATED — do not hand-edit. Source: moistlab/boards/orb_disc.py + orb_sheets.py; regenerate with tools/gen_kicad.py" (exclude_from_sim no) (at 25.4 213.36 0) (effects (font (size 2.032 2.032)) (justify left)))
-	(text "Provenance: every rating on this sheet is [I] — vendor web copy or folklore. No transcription pass has happened." (exclude_from_sim no) (at 25.4 218.44 0) (effects (font (size 1.778 1.778)) (justify left)))
-	(text "Pin numbers are hidden on parts whose package pinout has NOT been transcribed. Only the 74AHCT125 shows its numbers." (exclude_from_sim no) (at 25.4 223.52 0) (effects (font (size 1.778 1.778)) (justify left)))
+	(text "Provenance: ratings are [I] vendor web copy unless the part's note cites a document number — [M] only with a citation (first: U5/OPT4048, TI SBOSA84, 2026-08-03)." (exclude_from_sim no) (at 25.4 218.44 0) (effects (font (size 1.778 1.778)) (justify left)))
+	(text "Pin numbers are hidden on parts whose package pinout has NOT been transcribed. Only the 74AHCT125 and the OPT4048 have earned theirs." (exclude_from_sim no) (at 25.4 223.52 0) (effects (font (size 1.778 1.778)) (justify left)))
 	(text "Counts on this sheet are recovered from the power arithmetic in orb_disc.py, not typed here: see prove_system_matches_power_model." (exclude_from_sim no) (at 25.4 228.6 0) (effects (font (size 1.778 1.778)) (justify left)))
 	(text "Every block is a sheet: TAKEOFF is 2/4, POST BASE is 3/4, ORB DISC is 4/4. The disc's physical layout is a separate .kicad_pcb." (exclude_from_sim no) (at 25.4 233.68 0) (effects (font (size 1.778 1.778)) (justify left)))
