File: public/lights/orb-2-post-base.kicad_sch (KiCad schematic)
At the start: 17 parts, among them U1 LMR16030, U2 74AHCT125

Commit message: solar: h1 solar, OPT4048 sensor, drafted CAD drawings, plain-language sync note
Co-Authored-By: Claude Fable 5 <noreply@anthropic.com>
Claude-Session: https://claude.ai/code/session_01KGs7HAmqeyDzRmkLXBVjfP
Other:
- note added: "I2C up the riser to the sensors in the globes."
- note added: "Pin numbers are hidden on parts whose package pinout has NOT been transcribed. Only the 74AHCT125 and the OPT4048 have earned theirs."
- note added: "Provenance: ratings are [I] vendor web copy unless the part's note cites a document number — [M] only with a citation (first: U5/OPT4048, TI SBOSA84, 2026-08-03)."
- note added: "Pull-ups live here because the bus master does."
- note added: "The riser is ONE cable of 7 conductors to the FIRST disc;"
- note added: "the four discs daisy-chain from there. Drawn as four data lines"
- note added: "until the disc sheet's J1->J2 chain contradicted it."
- note removed: "I2C up the riser to the humidity sensor in the lowest globe. Pull-ups live here because the bus master does."
- note removed: "Pin numbers are hidden on parts whose package pinout has NOT been transcribed. Only the 74AHCT125 shows its numbers."
- note removed: "Provenance: every rating on this sheet is [I] — vendor web copy or folklore. No transcription pass has happened."
- note removed: "The riser is ONE cable of 7 conductors to the FIRST disc; the four discs daisy-chain from there. It was drawn as four data lines until the disc sheet's J1->J2 chain contradicted it."
