File: public/lights/orb-3-orb-disc.kicad_sch (KiCad schematic)
At the start: 26 parts, among them J1 5-pos 2.0 mm, J2 5-pos 2.0 mm, U1 AL8860, U2 LMR16030, U3 AL8860, U4 HDC3020

Commit message: solar: h1 solar, OPT4048 sensor, drafted CAD drawings, plain-language sync note
Co-Authored-By: Claude Fable 5 <noreply@anthropic.com>
Claude-Session: https://claude.ai/code/session_01KGs7HAmqeyDzRmkLXBVjfP
Parts:
- removed X_SKY: sky colour sensor - NO PART CHOSEN, symbol moistlab:GAP_SKY_SENSE
- added C_3V3: (1 uF 16 V X7R 0603), symbol moistlab:C
- added C_SKY: (100 nF 16 V X7R 0402), symbol moistlab:C
- added U5: OPT4048, symbol moistlab:OPT4048
- added U6: AP2112K-3.3, symbol moistlab:AP2112K-3.3
Connections:
- net +5V_LED: now also U6.1 (VIN), U6.3 (EN); no longer C_SHT.1, U4.1 (VDD)
- net GND: now also C_3V3.2, C_SKY.2, U5.2 (ADDR), U5.4 (GND), U6.2 (GND)
- net SCL: now also U5.5 (SCL)
- net SDA: now also U5.8 (SDA)
- new net +3V3_SNS: C_3V3.1, C_SHT.1, C_SKY.1, U4.1 (VDD), U5.1 (VDD), U6.5 (VOUT)
- no-connect marks 0 -> 3
Other:
- note added: "5 V buck PER DISC (base-fed 5 V loses a fifth in the riser); white strings 5s at 3.2 V worst-bin Vf under the 20 V floor."
- note added: "Disc is 70 mm through a 101.6 mm globe mount ID [M operator, corrected 2026-08-02]."
- note added: "Per disc [I]: white 4.80 W + pixels 5.12 W = 11.67 W at the bus; four discs + base = 48.6 W per post."
- note added: "Pin numbers are hidden on parts whose package pinout has NOT been transcribed. Only the 74AHCT125 and the OPT4048 have earned theirs."
- note added: "Provenance: ratings are [I] vendor web copy unless the part's note cites a document number — [M] only with a citation (first: U5/OPT4048, TI SBOSA84, 2026-08-03)."
- note added: "Same ten emitters, same 4.80 W — the second driver buys colour temperature."
- note added: "Sample window: one skipped frame - held by orb_program, not by this sheet."
- note added: "TWO white channels: 2200 K on U1, 3000 K on U3, 5s at 0.15 A each."
- note added: "The globe has to breathe: vent + weep + coating are the defences; U4 is how anyone knows they work (orb_climate.py)."
- note added: "U5 reads the sky THROUGH the globe (TI: characterized under dark cover glass), and only while every emitter is blanked."
- note removed: "Disc is 70 mm through a 101.6 mm globe bore [M operator]."
- note removed: "Each white string is 5s at 3.2 V worst-bin Vf = 16 V, plus 0.6 V driver headroom, under the 20 V bus floor."
- note removed: "Per disc [I]: white 4.80 W at the LEDs, pixels 5.12 W at the ring, 11.67 W at the bus after 85% conversion. Four discs + base = 48.6 W per post."
- note removed: "Pin numbers are hidden on parts whose package pinout has NOT been transcribed. Only the 74AHCT125 shows its numbers."
- note removed: "Provenance: every rating on this sheet is [I] — vendor web copy or folklore. No transcription pass has happened."
- note removed: "TWO white channels: 2200 K on U1 and 3000 K on U3, 5s each at 0.15 A. Same ten emitters and the same 4.80 W the single channel drew — what the second driver buys is colour temperature, not light."
- note removed: "The 5 V buck is PER DISC on purpose: a base-fed 5 V rail loses a fifth of itself in the riser before the first frame."
- note removed: "The globe has to breathe: an ePTFE vent, a weep path and a coated board are the defences; U4 is how anyone knows they work. See moistlab/boards/orb_climate.py."
- note removed: "X_SKY samples the sky THROUGH the globe, so it reads what the sphere shows - and only while every emitter is blanked. Window held by orb_program."
